File: hardware/badge-esp32-s3/sd_card.kicad_sch (KiCad schematic)
At the start: 0 parts

Commit message: Update sd_card.kicad_sch
Parts:
- added J4: Micro_SD_Card, symbol Connector:Micro_SD_Card
Connections:
- new net 3.3V: J4.4 (VDD)
- new net GND: J4.6 (VSS)
- new net MISO: J4.7 (DAT0)
- new net MOSI: J4.3 (CMD)
- new net SCLK: J4.5 (CLK)
- new net SD_CS: J4.2 (DAT3/CD)
- no-connect marks 0 -> 2

Commit message: Updated SD card sub schematic
Parts:
- added C14: 0.1uF, Capacitor_SMD:C_0603_1608Metric, symbol Device:C
Connections:
- net GND: now also J4.9 (SHIELD), C14.2
- net 3.3V renamed VCC
- net VCC: now also C14.1

Commit message: Updated SPI SD card Interface
Connections:
- net VCC renamed 3.3V
Changed lines of the file:
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@@
+		)
+	)
+	(hierarchical_label "3.3V"
+		(shape input)
+		(at 99.06 38.1 90)
+		(effects
+			(font
+				(size 1.27 1.27)
+			)
+			(justify left)
+		)
+	)
+	(hierarchical_label "3.3V"
+		(shape input)
+		(at 129.54 54.61 180)
+		(effects
+			(font
+				(size 1.27 1.27)
+			)
+			(justify right)
 		)
 	)
@@
 	)
 	(hierarchical_label "MISO"
-		(shape input)
+		(shape output)
 		(at 149.86 62.23 180)
 		(effects
@@
 			)
 			(justify right)
-		)
-	)
-	(symbol
-		(lib_id "power:VCC")
-		(at 129.54 54.61 90)
-		(unit 1)
-		(exclude_from_sim no)
-		(in_bom yes)
-		(on_board yes)
-		(dnp no)
-		(fields_autoplaced yes)
-		(property "Reference" "#PWR037"
-			(at 133.35 54.61 0)
-			(effects
-				(font
-					(size 1.27 1.27)
-				)
-				(hide yes)
-			)
-		)
-		(property "Value" "VCC"
-			(at 125.73 54.6099 90)
-			(effects
-				(font
-					(size 1.27 1.27)
-				)
-				(justify left)
-			)
-		)
-		(property "Footprint" ""
-			(at 129.54 54.61 0)
-			(effects
-				(font
-					(size 1.27 1.27)
-				)
-				(hide yes)
-			)
-		)
-		(property "Datasheet" ""
-			(at 129.54 54.61 0)
-			(effects
-				(font
-					(size 1.27 1.27)
-				)
-				(hide yes)
-			)
-		)
-		(property "Description" "Power symbol creates a global label with name \"VCC\""
-			(at 129.54 54.61 0)
-			(effects
-				(font
-					(size 1.27 1.27)
-				)
-				(hide yes)
-			)
-		)
-		(pin "1"
-		)
-		(instances
-			(project ""
-				(path "/e2af9a6c-dbe9-4de2-9ba6-ea213a7300ec/61971e93-08b4-4717-9ec8-ac07d8e404d2"
-					(reference "#PWR037")
-					(unit 1)
-				)
-			)
 		)
 	)
@@
 					(unit 1)
 				)
-			)
-		)
-	)
-	(symbol
-		(lib_id "power:VCC")
-		(at 99.06 38.1 0)
-		(unit 1)
-		(exclude_from_sim no)
-		(in_bom yes)
-		(on_board yes)
-		(dnp no)
-		(fields_autoplaced yes)
-		(property "Reference" "#PWR035"
-			(at 99.06 41.91 0)
-			(effects
-				(font
-					(size 1.27 1.27)
-				)
-				(hide yes)
-			)
-		)
-		(property "Value" "VCC"
-			(at 99.06 33.02 0)
-			(effects
-				(font
-					(size 1.27 1.27)
-				)
-			)
-		)
-		(property "Footprint" ""
-			(at 99.06 38.1 0)
-			(effects
-				(font
-					(size 1.27 1.27)
-				)
-				(hide yes)
-			)
-		)
-		(property "Datasheet" ""
-			(at 99.06 38.1 0)
-			(effects
-				(font
-					(size 1.27 1.27)
-				)
-				(hide yes)
-			)
-		)
-		(property "Description" "Power symbol creates a global label with name \"VCC\""
-			(at 99.06 38.1 0)
-			(effects
-				(font
-					(size 1.27 1.27)
-				)
-				(hide yes)
-			)
-		)
-		(pin "1"
-		)
-		(instances
-			(project ""
-				(path "/e2af9a6c-dbe9-4de2-9ba6-ea213a7300ec/61971e93-08b4-4717-9ec8-ac07d8e404d2"
-					(reference "#PWR035")
-					(unit 1)
-				)
