File: hardware/badge-esp32-s3/leds.kicad_sch (KiCad schematic)
At the start: 0 parts

Commit message: Push Buttons and Single Color LED
Parts:
- added D12: Red, PCM_JLCPCB:D_0603, symbol PCM_JLCPCB-Diodes:LED,0603,Red
- added R22: 51Ω, PCM_JLCPCB:R_0603, symbol PCM_JLCPCB-Resistors:0603,51Ω
Connections:
- new net: D12.2, R22.2
- new net 3.3vin: R22.1
- new net GND: D12.1
Other:
- note added: "Vf = 2.2V If = 20ma (3.3 - 2.2)/.02 = 55 ohms"
