File: hardware v4.0/badge-esp32-s3/minibadge.kicad_sch (KiCad schematic)
At the start: 15 parts, among them J12 Conn_01x02_Socket, J13 Conn_01x04_Socket, J5 Conn_01x02_Socket, J6 Conn_01x04_Socket, J7 Conn_01x08_Socket, J8 Conn_01x08_Socket, J9 Conn_02x06_Odd_Even

Commit message: started changes for 4.0.1
fixed footprint, joystick collision, Changed to Forced PWM mode for boost converter, Fixed some silkscreen errors
Parts:
- added C38, C39: 1uF, PCM_JLCPCB:C_0402, symbol PCM_JLCPCB-Capacitors:0402,1uF
Connections:
- net GND: now also C38.2, C39.2
- net VBAT: now also C38.1, C39.1

Commit message: added remainder of changes
Parts:
- J13, J6: LCSC C2718488 -> C18078127
Changed lines of the file:
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@@
 			)
 		)
-		(property "LCSC" "C2718488"
+		(property "LCSC" "C18078127"
 			(at 107.95 82.55 0)
 			(effects
@@
 			)
 		)
-		(property "LCSC" "C2718488"
+		(property "LCSC" "C18078127"
 			(at 165.1 82.55 0)
 			(effects
