File: hardware v4.0/badge-esp32-s3/badge-esp32-s3.kicad_sch (KiCad schematic)
At the start: 9 parts, among them U1 ESP32-S3-MINI-1-N4R2

Commit message: added 470R resistor to boot switch to prevent conflict
Other:
- sheet Download Mode Toggle: file pd_switch.kicad_sch -> dm_pd_switch.kicad_sch
Changed lines of the file:
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@@
 			)
 		)
-		(property "Sheetfile" "pd_switch.kicad_sch"
+		(property "Sheetfile" "dm_pd_switch.kicad_sch"
 			(at 209.55 27.2546 0)
 			(effects

Commit message: added DRD, 3.3V switching reg, and VIN
Other:
- sheet ESP USB: file usbc_5v_v2_data.kicad_sch -> usbc_esp_5v_v2_data.kicad_sch
- sheet USB-UART: file usbc_5v_v2_data.kicad_sch -> usbc_UART_5v_v2_data.kicad_sch
Changed lines of the file:
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@@
 			)
 		)
-		(property "Sheetfile" "usbc_5v_v2_data.kicad_sch"
+		(property "Sheetfile" "usbc_esp_5v_v2_data.kicad_sch"
 			(at 25.4 59.0046 0)
 			(effects
@@
 			)
 		)
-		(property "Sheetfile" "usbc_5v_v2_data.kicad_sch"
+		(property "Sheetfile" "usbc_UART_5v_v2_data.kicad_sch"
 			(at 245.11 53.9246 0)
 			(effects
