File: hardware v4.0/badge-esp32-s3/badge-esp32-s3.kicad_sch (KiCad schematic)
At the start: 9 parts, among them U1 ESP32-S3-MINI-1-N4R2

Commit message: finished schematics and layout
Parts:
- removed H5: MountingHole, MountingHole:MountingHole_5.3mm_M5, symbol Mechanical:MountingHole
- H1, H2, H3, H4: footprint MountingHole_3.2mm_M3_ISO7380_Pad_TopBottom -> misc-lib:MountingHole_3.2mm_M3_ISO7380_Pad_TopBottom
Other:
- sheet Charging renamed Power Input Managment
- sheet ESP USB ports: added 5V_stable, USB_RAW_HighCurrent, USB_RAW_LowCurrent; removed VBUS, VCC_5V
- sheet Exposed Pins ports: added none; removed IO45, IO46
- sheet Power Input Managment ports: added PWR_RAW, USB_HC, USB_LC; removed USB_5V, VOUT
- sheet USB-UART ports: added USB_RAW_HighCurrent, USB_RAW_LowCurrent; removed VCC_5V
- sheet Voltage Management ports: added PWR_RAW; removed VBATT, VCC_5V
- note removed: "Implied diode OR"
