File: hardware v4.0/badge-esp32-s3/usbc_esp_5v_v2_data.kicad_sch (KiCad schematic)
At the start: 17 parts, among them J2 Connector, USB-TYPE-C-16P, U10 PCA9536DGKR, U11 SY6288F1ABC, U12 SY6288F1ABC, U8 TUSB321AIRWBR

Commit message: break before make circuit
Parts:
- removed R66: 20kΩ, PCM_JLCPCB:R_0402, symbol PCM_JLCPCB-Resistors:0402,20kΩ
- removed U10: PCA9536DGKR, lcsc-lib:VSSOP-8_L3.0-W3.0-P0.65-LS4.9-BL, symbol lcsc-lib:PCA9536DGKR
- added C3, C4: 100nF, PCM_JLCPCB:C_0402, symbol PCM_JLCPCB-Capacitors:0402,100nF
- added D9: BAT54W_C7502705, lcsc-lib:SOD-123_L2.7-W1.6-LS3.7-RD, symbol lcsc-lib:BAT54W_C7502705
- added Q10: AO3424, lcsc-lib:SC-59-3_L2.9-W1.6-P0.95-LS2.9-BR, symbol lcsc-lib:AO3424
- added R66, R69, R70: 10kΩ, PCM_JLCPCB:R_0402, symbol PCM_JLCPCB-Resistors:0402,10kΩ
Connections:
- net Boost_5V: now also R69.1
- net GND: now also C3.2, C4.2, Q10.2 (S)
- net USB_ID: now also D9.1 (K), R66.1
- net USB_SINK_EN: now also C3.1, D9.2 (A), R70.2
- net USB_SOURCE_EN: now also C4.1, Q10.3 (D), R69.2
- net VBUS: now also R70.1
- net PORT: no longer names the net of U8.4 (PORT)
- new net: Q10.1 (G), R66.2
- no-connect marks 8 -> 9
Other:
- note added: "Break Before Make Control"
- note removed: "For firmware dev: (Break before make) When sourcing power to an external USB device Turn OFF USB sink load switch then turn ON the USB source load switch. If this is not respected ustable power feedback loops may occur."
- note removed: "Interface via I2C expander"
- note removed: "PORT tells the TUSB321AIRWBR what to adversise our device as (PWR source (High), PWR sink (LOW), or DRD (HI-Z)). If automatic roles (or DRD) is desired configure this as an input so the chip sees a HI-Z state. Configuring PORT as a DRD is the standard option."
