File: hardware v4.0/badge-esp32-s3/leds.kicad_sch (KiCad schematic)
At the start: 33 parts

Commit message: finished schematics and layout
Parts:
- removed AL1, AL10, AL11, AL12, AL13, AL14, AL15, AL16, AL17, AL18, AL19, AL2, AL20, AL21, AL22, AL23, AL24, AL3, AL4, AL5, AL6, AL7, AL8, AL9: ~, lcsc-lib:LED-SMD_6P-L2.2-W2.2-TL-1, symbol lcsc-lib:WS2813B-2121
- removed C42: GVS1A107M0604CN, lcsc-lib:CAP-SMD_BD6.3-L6.6-W6.6-LS7.3-FD, symbol lcsc-lib:GVS1A107M0604CN
- removed R19: 5.1kΩ, PCM_JLCPCB:R_0402, symbol PCM_JLCPCB-Resistors:0402,5.1kΩ
- removed R20: 100Ω, PCM_JLCPCB:R_0402, symbol PCM_JLCPCB-Resistors:0402,100Ω
- removed R21, R22: 47Ω, PCM_JLCPCB:R_0402, symbol PCM_JLCPCB-Resistors:0402,47Ω
- added AL1, AL10, AL11, AL12, AL13, AL14, AL15, AL16, AL17, AL18, AL19, AL2, AL20, AL21, AL22, AL23, AL24, AL3, AL4, AL5, AL6, AL7, AL8, AL9: SK6805MICRO-J, lcsc-lib:LED-SMD_4P-SK6805MICRO-J, symbol lcsc-lib:SK6805MICRO-J
- added R19, R20: 680Ω, PCM_JLCPCB:R_0402, symbol PCM_JLCPCB-Resistors:0402,680Ω
- added R21: 1.2kΩ, PCM_JLCPCB:R_0402, symbol PCM_JLCPCB-Resistors:0402,1.2kΩ
- added R22: 300Ω, PCM_JLCPCB:R_0402, symbol PCM_JLCPCB-Resistors:0402,300Ω
- added R68: 10kΩ, PCM_JLCPCB:R_0402, symbol PCM_JLCPCB-Resistors:0402,10kΩ
Connections:
- net 5V: now also AL1.4 (VDD), AL10.4 (VDD), AL11.4 (VDD), AL12.4 (VDD), AL13.4 (VDD), AL14.4 (VDD), AL15.4 (VDD), AL16.4 (VDD), AL17.4 (VDD), AL18.4 (VDD), AL19.4 (VDD), AL2.4 (VDD), AL20.4 (VDD), AL21.4 (VDD), AL22.4 (VDD), AL23.4 (VDD), AL24.4 (VDD), AL3.4 (VDD), AL4.4 (VDD), AL5.4 (VDD), AL6.4 (VDD), AL7.4 (VDD), AL8.4 (VDD), AL9.4 (VDD)
- net AddrLED: now also AL1.3 (DIN), R68.1
- net GND: now also AL1.2 (VSS), AL10.2 (VSS), AL11.2 (VSS), AL12.2 (VSS), AL13.2 (VSS), AL14.2 (VSS), AL15.2 (VSS), AL16.2 (VSS), AL17.2 (VSS), AL18.2 (VSS), AL19.2 (VSS), AL2.2 (VSS), AL20.2 (VSS), AL21.2 (VSS), AL22.2 (VSS), AL23.2 (VSS), AL24.2 (VSS), AL3.2 (VSS), AL4.2 (VSS), AL5.2 (VSS), AL6.2 (VSS), AL7.2 (VSS), AL8.2 (VSS), AL9.2 (VSS), R19.2, R20.2, R21.2, R68.2
- net LED_SINGLE1: now also R22.1
- net at LED1.1 (-): now also R20.1
- net at LED1.2 (-): now also R21.1
- net at LED1.3 (-): now also R19.1
- net at D14.2: now also R22.2
- new net: AL2.1 (DOUT), AL3.3 (DIN)
- new net: AL1.1 (DOUT), AL2.3 (DIN)
- new net: AL15.1 (DOUT), AL16.3 (DIN)
- new net: AL19.1 (DOUT), AL20.3 (DIN)
- new net: AL18.1 (DOUT), AL19.3 (DIN)
- new net: AL23.1 (DOUT), AL24.3 (DIN)
- new net: AL22.1 (DOUT), AL23.3 (DIN)
- new net: AL7.1 (DOUT), AL8.3 (DIN)
- new net: AL21.1 (DOUT), AL22.3 (DIN)
- new net: AL20.1 (DOUT), AL21.3 (DIN)
- new net: AL17.1 (DOUT), AL18.3 (DIN)
- new net: AL6.1 (DOUT), AL7.3 (DIN)
- new net: AL10.1 (DOUT), AL11.3 (DIN)
- new net: AL10.3 (DIN), AL9.1 (DOUT)
- new net: AL3.1 (DOUT), AL4.3 (DIN)
- new net: AL5.1 (DOUT), AL6.3 (DIN)
- new net: AL4.1 (DOUT), AL5.3 (DIN)
- new net: AL14.1 (DOUT), AL15.3 (DIN)
- new net: AL11.1 (DOUT), AL12.3 (DIN)
- new net: AL13.1 (DOUT), AL14.3 (DIN)
- new net: AL12.1 (DOUT), AL13.3 (DIN)
- new net AL16_OUT: AL16.1 (DOUT), AL17.3 (DIN)
- new net AL8_OUT: AL8.1 (DOUT), AL9.3 (DIN)
- no-connect marks 2 -> 1
Other:
- note removed: "Vf = 2.2V If = 20ma (3.3 - 2.2)/.02 = 55 ohms"
