File: hardware v4.0/badge-esp32-s3/usbc_UART_5v_v2_data.kicad_sch (KiCad schematic)
At the start: 8 parts, among them J1 Connector, USB-TYPE-C-16P

Commit message: finished schematics and layout
Parts:
- added D17: SS32F_C719168, lcsc-lib:SMAF_L3.5-W2.6-LS4.7-RD, symbol lcsc-lib:SS32F_C719168
Connections:
- net VBUS: now also C5.1, D17.2 (A)
- net VCC_5V renamed USB_RAW_LowCurrent
- net USB_RAW_LowCurrent: no longer C5.1
- new net USB_RAW_HighCurrent: D17.1 (K)
Other:
- moved on the sheet: D5
Changed lines of the file:
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@@
+	)
+	(junction
+		(at 166.37 60.96)
+		(diameter 0)
+		(color 0 0 0 0)
 	)
 	(junction
@@
 	)
 	(junction
-		(at 166.37 60.96)
-		(diameter 0)
-		(color 0 0 0 0)
-	)
-	(junction
 		(at 151.13 60.96)
 		(diameter 0)
@@
 	(wire
 		(pts
+			(xy 186.69 49.53) (xy 198.12 49.53)
+		)
+		(stroke
+			(width 0)
+			(type default)
+		)
+	)
+	(wire
+		(pts
 			(xy 124.46 76.2) (xy 142.24 76.2)
 		)
@@
 	(wire
 		(pts
-			(xy 151.13 60.96) (xy 154.94 60.96)
-		)
-		(stroke
-			(width 0)
-			(type default)
-		)
-	)
-	(wire
-		(pts
-			(xy 172.72 60.96) (xy 166.37 60.96)
+			(xy 151.13 60.96) (xy 166.37 60.96)
+		)
+		(stroke
+			(width 0)
+			(type default)
+		)
+	)
+	(wire
+		(pts
+			(xy 166.37 49.53) (xy 179.07 49.53)
 		)
 		(stroke
@@
 	(wire
 		(pts
-			(xy 162.56 60.96) (xy 166.37 60.96)
+			(xy 187.96 60.96) (xy 198.12 60.96)
 		)
 		(stroke
@@
 	(wire
 		(pts
+			(xy 166.37 60.96) (xy 166.37 49.53)
+		)
+		(stroke
+			(width 0)
+			(type default)
+		)
+	)
+	(wire
+		(pts
 			(xy 129.54 110.49) (xy 129.54 100.33)
 		)
@@
 		(pts
 			(xy 129.54 87.63) (xy 129.54 81.28)
+		)
+		(stroke
+			(width 0)
+			(type default)
+		)
+	)
+	(wire
+		(pts
+			(xy 166.37 60.96) (xy 177.8 60.96)
 		)
 		(stroke
@@
 		)
 	)
+	(hierarchical_label "USB_RAW_LowCurrent"
+		(shape bidirectional)
+		(at 198.12 49.53 0)
+		(effects
+			(font
+				(size 1.27 1.27)
+			)
+			(justify left)
+		)
+	)
 	(hierarchical_label "USBD_N"
 		(shape bidirectional)
@@
 		)
 	)
-	(hierarchical_label "VCC_5V"
+	(hierarchical_label "USB_RAW_HighCurrent"
 		(shape bidirectional)
-		(at 172.72 60.96 0)
+		(at 198.12 60.96 0)
 		(effects
 			(font
@@
 	)
 	(symbol
+		(lib_id "lcsc-lib:SS32F_C719168")
+		(at 182.88 60.96 180)
+		(unit 1)
+		(exclude_from_sim no)
+		(in_bom yes)
+		(on_board yes)
+		(dnp no)
+		(fields_autoplaced yes)
+		(property "Reference" "D17"
+			(at 182.88 54.61 0)
+			(effects
+				(font
+					(size 1.27 1.27)
+				)
+			)
+		)
+		(property "Value" "SS32F_C719168"
+			(at 182.88 57.15 0)
+			(effects
+				(font
+					(size 1.27 1.27)
+				)
+			)
+		)
+		(property "Footprint" "lcsc-lib:SMAF_L3.5-W2.6-LS4.7-RD"
+			(at 182.88 53.34 0)
+			(effects
+				(font
+					(size 1.27 1.27)
+				)
+				(hide yes)
+			)
+		)
+		(property "Datasheet" "https://lcsc.com/product-detail/Schottky-Barrier-Diodes-SBD_Shikues-SS32F_C719168.html"
+			(at 182.88 50.8 0)
+			(effects
+				(font
+					(size 1.27 1.27)
+				)
+				(hide yes)
+			)
+		)
+		(property "Description" ""
+			(at 182.88 60.96 0)
+			(effects
+				(font
+					(size 1.27 1.27)
+				)
+				(hide yes)
+			)
+		)
+		(property "Manufacturer" "SHIKUES(时科)"
+			(at 182.88 48.26 0)
+			(effects
+				(font
+					(size 1.27 1.27)
+				)
+				(hide yes)
+			)
+		)
+		(property "MPN" "SS32F"
+			(at 182.88 45.72 0)
+			(effects
+				(font
+					(size 1.27 1.27)
+				)
+				(hide yes)
+			)
+		)
+		(property "LCSC Part" "C719168"
+			(at 182.88 43.18 0)
+			(effects
+				(font
+					(size 1.27 1.27)
+				)
+				(hide yes)
+			)
+		)
+		(pin "2"
+		)
+		(pin "1"
+		)
+		(instances
+			(project "badge-esp32-s3"
+				(path "/e2af9a6c-dbe9-4de2-9ba6-ea213a7300ec/e365f6ed-f2b4-4ac9-8336-75c01e8e2e23"
+					(reference "D17")
+					(unit 1)
+				)
+			)
+		)
+	)
+	(symbol
 		(lib_id "PCM_JLCPCB-Diodes:Schottky,B0520W")
-		(at 158.75 60.96 90)
+		(at 182.88 49.53 90)
 		(unit 1)
 		(exclude_from_sim no)
@@
 		(fields_autoplaced yes)
 		(property "Reference" "D5"
-			(at 159.0675 54.61 90)
+			(at 183.1975 43.18 90)
 			(effects
 				(font
@@
 		)
 		(property "Value" "B0520W"
-			(at 159.0675 57.15 90)
+			(at 183.1975 45.72 90)
 			(effects
 				(font
@@
 		)
 		(property "Footprint" "PCM_JLCPCB:D_SOD-123"
-			(at 158.75 62.738 90)
+			(at 182.88 51.308 90)
 			(effects
 				(font
@@
 		)
 		(property "Datasheet" "https://wmsc.lcsc.com/wmsc/upload/file/pdf/v2/lcsc/2308281443_hongjiacheng-B0520W_C7502707.pdf"
-			(at 158.75 60.96 0)
+			(at 182.88 49.53 0)
 			(effects
 				(font
@@
 		)
 		(property "Description" "20V Independent Type 385mV@500mA 500mA SOD-123 Schottky Diodes ROHS"
-			(at 158.75 60.96 0)
+			(at 182.88 49.53 0)
 			(effects
 				(font
@@
 		)
 		(property "LCSC" "C7502707"
-			(at 158.75 60.96 0)
+			(at 182.88 49.53 0)
 			(effects
 				(font
@@
 		)
 		(property "Stock" "16019"
-			(at 158.75 60.96 0)
+			(at 182.88 49.53 0)
 			(effects
 				(font
@@
 		)
 		(property "Price" "0.020USD"
-			(at 158.75 60.96 0)
+			(at 182.88 49.53 0)
 			(effects
 				(font
@@
 		)
 		(property "Process" "SMT"
-			(at 158.75 60.96 0)
+			(at 182.88 49.53 0)
 			(effects
 				(font
@@
 		)
 		(property "Minimum Qty" "15"
-			(at 158.75 60.96 0)
+			(at 182.88 49.53 0)
 			(effects
 				(font
@@
 		)
 		(property "Attrition Qty" "4"
-			(at 158.75 60.96 0)
+			(at 182.88 49.53 0)
 			(effects
 				(font
@@
 		)
 		(property "Class" "Preferred Component"
-			(at 158.75 60.96 0)
+			(at 182.88 49.53 0)
 			(effects
 				(font
@@
 		)
 		(property "Category" "Diodes,Schottky Barrier Diodes (SBD)"
-			(at 158.75 60.96 0)
+			(at 182.88 49.53 0)
 			(effects
 				(font
@@
 		)
 		(property "Manufacturer" "hongjiacheng"
-			(at 158.75 60.96 0)
+			(at 182.88 49.53 0)
 			(effects
 				(font
@@
 		)
 		(property "Part" "B0520W"
-			(at 158.75 60.96 0)
-			(effects
-				(font
+			(at 182.88 49.53 0)
+			(effects
+				(font
