File: hardware v4.0/badge-esp32-s3/badge-esp32-s3.kicad_pcb (KiCad board)
At the start: 2 copper layers, 131.5 x 83.5 mm, 185 parts, among them CN1 B4B-PH-SM4-TB (LF)(SN), J1 Connector, USB-TYPE-C-16P, J11 Conn_02x03_Odd_Even, J12 Conn_01x02_Socket, J13 Conn_01x04_Socket, J14 Conn_01x02_Socket, J15 Conn_01x02_Socket, J2 Connector, USB-TYPE-C-16P, J3 Conn_02x06_Odd_Even, J4 Conn_02x15_Odd_Even, J5 Conn_01x02_Socket, J6 Conn_01x04_Socket, J7 Conn_01x08_Socket, J8 Conn_01x08_Socket, J9 Conn_02x06_Odd_Even, P1 PH-2A_C2319, P2 FPC 0.5MM 12P Pull type H2.0m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, Q1 SS8050 200-350, Q2 SS8050 200-350, Q3 HL2301A, Q4 HL2301A, Q5 DTC114E, Q6 AO3424, Q7 AO3424, SW1 TS-1088-AR02016, SW2 TS-1088-AR02016, SW4 TS665CJ, SW5 TS665CJ, SW6 TS665CJ, SW7 TS665CJ, SW8 TS665CJ, SW9 TS665CJ, U1 ESP32-S3-MINI-1-N4R2, U18 MMA8452QR1_C11360, U2 TPS630701RNMR, U3 CP2102N-A02-GQFN28R, U4 TP4056, U6 ZX-SH1.0-4PWT, U7 HS20HS072RX-fpc, U8 TLV75733PDBVR

Commit message: finished schematics and layout
Parts:
- removed D11: B0520W, PCM_JLCPCB:D_SOD-123
- removed the G*** at (104.5, 137.1)
- removed H5: MountingHole, MountingHole:MountingHole_5.3mm_M5
- removed Power1: SK-12F04-G050, lcsc-lib:SW-TH_G-SWITCH_SK-12F04-G050
- removed Q4: HL2301A, PCM_JLCPCB:Q_SOT-23
- removed Q7: AO3424, lcsc-lib:SC-59-3_L2.9-W1.6-P0.95-LS2.9-BR
- removed R2: 5.1kΩ, PCM_JLCPCB:R_0402
- added C24: 10uF, PCM_JLCPCB:C_0603, F.Cu at (203.5, 96.3)
- added C38: 22uF, PCM_JLCPCB:C_0805, F.Cu at (193.4, 115.1)
- added C39: 10uF, PCM_JLCPCB:C_0603, F.Cu at (193.3, 105.0)
- added C40: 22uF, PCM_JLCPCB:C_0805, F.Cu at (183.8, 103.1)
- added C41: 100nF, PCM_JLCPCB:C_0402, F.Cu at (196.8, 106.7)
- added C44: 100nF, PCM_JLCPCB:C_0402, F.Cu at (189.7, 117.0)
- added D10: B5819WT, PCM_JLCPCB:D_SOD-523, F.Cu at (176.8, 76.7)
- added D16: B0520W, PCM_JLCPCB:D_SOD-123, F.Cu at (185.9, 65.8)
- added D17: SS32F_C719168, lcsc-lib:SMAF_L3.5-W2.6-LS4.7-RD, F.Cu at (182.4, 65.2)
- added D18: SS32F_C719168, lcsc-lib:SMAF_L3.5-W2.6-LS4.7-RD, F.Cu at (182.9, 70.8)
- added D19: Red, PCM_JLCPCB:D_0603, F.Cu at (178.7, 75.4)
- added D20: BZT52-B5V1S, lcsc-lib:SOD-323_L1.8-W1.3-LS2.5-RD, F.Cu at (198.8, 108.4)
- added D21: BZT52-B5V1S, lcsc-lib:SOD-323_L1.8-W1.3-LS2.5-RD, F.Cu at (198.9, 102.0)
- added L1: ANR4030T3R9M, lcsc-lib:IND-SMD_L4.0-W4.0, F.Cu at (186.1, 115.4)
- added L2: MPZ2012S101AT000, lcsc-lib:L0805, F.Cu at (194.8, 111.4)
- added P3: WJ124-3.81-2P, lcsc-lib:CONN-TH_2P-P3.81_KF124-3.81-2P, F.Cu at (207.5, 87.6)
- added Q10: DMN3150L-7, lcsc-lib:SOT-23-3_L2.9-W1.6-P1.90-LS2.8-BR-CW, F.Cu at (195.0, 97.7)
- added Q11: DMN3150L-7, lcsc-lib:SOT-23-3_L2.9-W1.6-P1.90-LS2.8-BR-CW, F.Cu at (199.4, 97.8)
- added R56: 100kΩ, PCM_JLCPCB:R_0402, F.Cu at (183.7, 95.8)
- added R57: 68kΩ, PCM_JLCPCB:R_0402, F.Cu at (201.2, 106.6)
- added R58: 47kΩ, PCM_JLCPCB:R_0402, F.Cu at (196.8, 104.7)
- added R59: 1MΩ, PCM_JLCPCB:R_0402, F.Cu at (201.2, 108.7)
- added R61: 3.3kΩ, PCM_JLCPCB:R_0402, F.Cu at (181.4, 78.5)
- added R62: 100kΩ, PCM_JLCPCB:R_0402, F.Cu at (201.2, 104.7)
- added R64: 330Ω, PCM_JLCPCB:R_0402, F.Cu at (177.0, 74.1)
- added R65: 12kΩ, PCM_JLCPCB:R_0402, F.Cu at (177.3, 71.6)
- added R66: 10kΩ, PCM_JLCPCB:R_0402, F.Cu at (175.5, 76.6)
- added R68: 10kΩ, PCM_JLCPCB:R_0402, F.Cu at (104.3, 141.3)
- added R69: 10kΩ, PCM_JLCPCB:R_0402, F.Cu at (177.0, 75.0)
- added R70: 10kΩ, PCM_JLCPCB:R_0402, F.Cu at (176.3, 78.5)
- added R71: 470kΩ, PCM_JLCPCB:R_0402, F.Cu at (201.2, 102.8)
- added SW10: SK22D02G5, lcsc-lib:SW-TH_SK22D02G5, F.Cu at (208.1, 102.1)
- added U11: SY6288F1ABC, lcsc-lib:SOT-23-6_L2.9-W1.6-P0.95-LS2.8-BL, F.Cu at (181.9, 76.0)
- added U12: SY6288F1ABC, lcsc-lib:SOT-23-6_L2.9-W1.6-P0.95-LS2.8-BL, F.Cu at (179.6, 72.1)
- added U5: TPS2121RUXR, lcsc-lib:VQFN-HR-12_L2.5-W2.0-P0.50-BL, F.Cu at (198.8, 105.6)
- added U9: AP63203WU-7, lcsc-lib:TSOT-26_L2.9-W1.6-P0.95-LS2.8-BL, F.Cu at (190.6, 114.8)
- AL1, AL10, AL11, AL12, AL13, AL14, AL15, AL16, AL17, AL18, AL19, AL2, AL20, AL21, AL22, AL23, AL24, AL3, AL4, AL5, AL6, AL7, AL8, AL9: value ~ -> SK6805MICRO-J; footprint lcsc-lib:LED-SMD_6P-L2.2-W2.2-TL-1 -> lcsc-lib:LED-SMD_4P-SK6805MICRO-J
- C28: value TMK107BBJ106MA-T -> 22uF; footprint lcsc-lib:C0603 -> PCM_JLCPCB:C_0805
- C29, C30, C31: footprint lcsc-lib:C0805 -> PCM_JLCPCB:C_0805
- C3, C4: value 1uF -> 100nF
- D9: value B0520W -> BZT52-B10S-PEC; footprint PCM_JLCPCB:D_SOD-123 -> lcsc-lib:SOD-323_L1.8-W1.3-LS2.5-RD-1
- H1, H2, H3, H4: footprint MountingHole:MountingHole_3.2mm_M3_ISO7380_Pad_TopBottom -> misc-lib:MountingHole_3.2mm_M3_ISO7380_Pad_TopBottom
- Q3: value HL2301A -> AP1606; footprint PCM_JLCPCB:Q_SOT-23 -> lcsc-lib:DFN-3L_L1.0-W0.6-P0.65-BR
- Q6: value AO3424 -> SI2301CDS-T1-GE3; footprint lcsc-lib:SC-59-3_L2.9-W1.6-P0.95-LS2.9-BR -> lcsc-lib:SOT-23-3_L3.0-W1.7-P0.95-LS2.9-BR
- R19: value 5.1kΩ -> 680Ω
- R20: value 100Ω -> 680Ω
- R21: value 47Ω -> 1.2kΩ
- R22: value 47Ω -> 300Ω
- R24, R48: value 100kΩ -> 1MΩ
- R44: value 100kΩ -> 10kΩ
- R46: value 47kΩ -> 10kΩ
- R5: value 5.1kΩ -> 910k; footprint PCM_JLCPCB:R_0402 -> lcsc-lib:R0402
- R54: value 10kΩ -> 300Ω
- R6: value 5.1kΩ -> 10kΩ
- U8: value TLV75733PDBVR -> TUSB321AIRWBR; footprint lcsc-lib:SOT-23-5_L2.9-W1.6-P0.95-LS2.8-BL -> lcsc-lib:X2QFN-12_L1.6-W1.6-P0.40-BL
- moved D5 74.9 mm to (185.7, 62.1), turned to 180 degrees
- moved R41 46.3 mm to (192.2, 135.4)
- moved C34 46.0 mm to (191.2, 137.1)
- moved R44 44.3 mm to (190.2, 137.1), turned to -90 degrees
- moved D9 43.5 mm to (201.9, 97.8), turned to -90 degrees
- moved Q3 32.9 mm to (174.4, 77.3)
- moved U8 24.1 mm to (173.1, 75.5), turned to 180 degrees
- moved C4 19.3 mm to (173.9, 78.5), turned to 180 degrees
- moved C3 19.1 mm to (178.1, 78.1), turned to -90 degrees
- moved R54 18.7 mm to (203.4, 108.2), turned to 90 degrees
- moved D1 17.3 mm to (203.4, 102.2), turned to -90 degrees
- moved C11 17.0 mm to (181.0, 84.0), turned to 0 degrees
- moved C10 16.5 mm to (181.0, 85.3), turned to 0 degrees
- moved R42 15.7 mm to (164.4, 83.8)
- moved BUZZER1 14.8 mm to (162.1, 80.4)
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Connections:
- AL1 pad 1: GND -> Net-(AL1-DOUT)
- AL1 pad 2: /AddrLedMid -> GND
- AL1 pad 3: /5V_stable -> /AddrLedMid
- AL1 pad 4: Net-(AL1-DO) -> /5V_stable
- AL10 pad 1: /LEDs/BO_AL9 -> Net-(AL10-DOUT)
- AL10 pad 2: /LEDs/DO_AL9 -> GND
- AL10 pad 3: /5V_stable -> Net-(AL10-DIN)
- AL10 pad 4: Net-(AL10-DO) -> /5V_stable
- AL11 pad 1: Net-(AL10-BO) -> Net-(AL11-DOUT)
- AL11 pad 2: Net-(AL10-DO) -> GND
- AL11 pad 3: /5V_stable -> Net-(AL10-DOUT)
- AL11 pad 4: Net-(AL11-DO) -> /5V_stable
- AL12 pad 1: Net-(AL11-BO) -> Net-(AL12-DOUT)
- AL12 pad 2: Net-(AL11-DO) -> GND
- AL12 pad 3: /5V_stable -> Net-(AL11-DOUT)
- AL12 pad 4: Net-(AL12-DO) -> /5V_stable
- AL13 pad 1: Net-(AL12-BO) -> Net-(AL13-DOUT)
- AL13 pad 2: Net-(AL12-DO) -> GND
- AL13 pad 3: /5V_stable -> Net-(AL12-DOUT)
- AL13 pad 4: Net-(AL13-DO) -> /5V_stable
- AL14 pad 1: Net-(AL13-BO) -> Net-(AL14-DOUT)
- AL14 pad 2: Net-(AL13-DO) -> GND
- AL14 pad 3: /5V_stable -> Net-(AL13-DOUT)
- AL14 pad 4: Net-(AL14-DO) -> /5V_stable
- AL15 pad 1: Net-(AL14-BO) -> Net-(AL15-DOUT)
- AL15 pad 2: Net-(AL14-DO) -> GND
- AL15 pad 3: /5V_stable -> Net-(AL14-DOUT)
- AL15 pad 4: Net-(AL15-DO) -> /5V_stable
- AL16 pad 1: Net-(AL15-BO) -> /LEDs/AL16_OUT
- AL16 pad 2: Net-(AL15-DO) -> GND
- AL16 pad 3: /5V_stable -> Net-(AL15-DOUT)
- AL16 pad 4: Net-(AL16-DO) -> /5V_stable
- AL17 pad 1: Net-(AL16-BO) -> Net-(AL17-DOUT)
- AL17 pad 2: Net-(AL16-DO) -> GND
- AL17 pad 3: /5V_stable -> /LEDs/AL16_OUT
- AL17 pad 4: Net-(AL17-DO) -> /5V_stable
- AL18 pad 1: Net-(AL17-BO) -> Net-(AL18-DOUT)
- AL18 pad 2: Net-(AL17-DO) -> GND
- AL18 pad 3: /5V_stable -> Net-(AL17-DOUT)
- AL18 pad 4: /LEDs/DO_AL18 -> /5V_stable
- AL19 pad 1: /LEDs/BO_AL18 -> Net-(AL19-DOUT)
- AL19 pad 2: /LEDs/DO_AL18 -> GND
- AL19 pad 3: /5V_stable -> Net-(AL18-DOUT)
- AL19 pad 4: Net-(AL19-DO) -> /5V_stable
- AL2 pad 1: Net-(AL1-BO) -> Net-(AL2-DOUT)
- AL2 pad 2: Net-(AL1-DO) -> GND
- AL2 pad 3: /5V_stable -> Net-(AL1-DOUT)
- AL2 pad 4: Net-(AL2-DO) -> /5V_stable
- AL20 pad 1: Net-(AL19-BO) -> Net-(AL20-DOUT)
- AL20 pad 2: Net-(AL19-DO) -> GND
- AL20 pad 3: /5V_stable -> Net-(AL19-DOUT)
- AL20 pad 4: Net-(AL20-DO) -> /5V_stable
- AL21 pad 1: Net-(AL20-BO) -> Net-(AL21-DOUT)
- AL21 pad 2: Net-(AL20-DO) -> GND
- AL21 pad 3: /5V_stable -> Net-(AL20-DOUT)
- AL21 pad 4: Net-(AL21-DO) -> /5V_stable
- AL22 pad 1: Net-(AL21-BO) -> Net-(AL22-DOUT)
- AL22 pad 2: Net-(AL21-DO) -> GND
- AL22 pad 3: /5V_stable -> Net-(AL21-DOUT)
- AL22 pad 4: Net-(AL22-DO) -> /5V_stable
- AL23 pad 1: Net-(AL22-BO) -> Net-(AL23-DOUT)
- AL23 pad 2: Net-(AL22-DO) -> GND
- AL23 pad 3: /5V_stable -> Net-(AL22-DOUT)
- AL23 pad 4: Net-(AL23-DO) -> /5V_stable
- AL24 pad 1: Net-(AL23-BO) -> unconnected-(AL24-DOUT-Pad1)
- AL24 pad 2: Net-(AL23-DO) -> GND
- AL24 pad 3: /5V_stable -> Net-(AL23-DOUT)
- AL24 pad 4: unconnected-(AL24-DO-Pad4) -> /5V_stable
- AL3 pad 1: Net-(AL2-BO) -> Net-(AL3-DOUT)
- AL3 pad 2: Net-(AL2-DO) -> GND
- AL3 pad 3: /5V_stable -> Net-(AL2-DOUT)
- AL3 pad 4: Net-(AL3-DO) -> /5V_stable
- AL4 pad 1: Net-(AL3-BO) -> Net-(AL4-DOUT)
- AL4 pad 2: Net-(AL3-DO) -> GND
- AL4 pad 3: /5V_stable -> Net-(AL3-DOUT)
- AL4 pad 4: Net-(AL4-DO) -> /5V_stable
- AL5 pad 1: Net-(AL4-BO) -> Net-(AL5-DOUT)
- AL5 pad 2: Net-(AL4-DO) -> GND
- AL5 pad 3: /5V_stable -> Net-(AL4-DOUT)
- AL5 pad 4: Net-(AL5-DO) -> /5V_stable
- AL6 pad 1: Net-(AL5-BO) -> Net-(AL6-DOUT)
- AL6 pad 2: Net-(AL5-DO) -> GND
- AL6 pad 3: /5V_stable -> Net-(AL5-DOUT)
- AL6 pad 4: Net-(AL6-DO) -> /5V_stable
- AL7 pad 1: Net-(AL6-BO) -> Net-(AL7-DOUT)
- AL7 pad 2: Net-(AL6-DO) -> GND
- AL7 pad 3: /5V_stable -> Net-(AL6-DOUT)
- AL7 pad 4: Net-(AL7-DO) -> /5V_stable
- AL8 pad 1: Net-(AL7-BO) -> /LEDs/AL8_OUT
- AL8 pad 2: Net-(AL7-DO) -> GND
- AL8 pad 3: /5V_stable -> Net-(AL7-DOUT)
- AL8 pad 4: Net-(AL8-DO) -> /5V_stable
- AL9 pad 1: Net-(AL8-BO) -> Net-(AL10-DIN)
- AL9 pad 2: Net-(AL8-DO) -> GND
- AL9 pad 3: /5V_stable -> /LEDs/AL8_OUT
- AL9 pad 4: /LEDs/DO_AL9 -> /5V_stable
- C12 pad 1: /USB_5V -> /USB_LC
- C28 pad 1: GND -> +3.3V
- C28 pad 2: PWR_RAW -> GND
- C29 pad 1: GND -> +3.3V
- C29 pad 2: /5V_stable -> GND
- C3 pad 1: PWR_RAW -> /ESP USB/USB_SINK_EN
- C30 pad 1: GND -> /5V_stable
- C30 pad 2: /5V_stable -> GND
- C31 pad 1: GND -> /5V_stable
- C31 pad 2: /5V_stable -> GND
- C4 pad 1: +3.3V -> /ESP USB/USB_SOURCE_EN
- C5 pad 1: /USB_5V -> /VBUS
- C6 pad 1: /USB_5V -> /ESP USB/VBUS
- D12 pad 2: /USB_5V -> /USB_LC
- D5 pad 1: /USB_5V -> /USB_LC
- D8 pad 2: /VBUSB -> /ESP USB/VBUS
- D9 pad 1: /USB_5V -> Net-(D9-C)
- D9 pad 2: /VBUSB -> GND
- J2 pad A5: Net-(J2-CC1) -> /ESP USB/CC1
- J2 pad A9B4: /VBUSB -> /ESP USB/VBUS
- J2 pad B5: Net-(J2-CC2) -> /ESP USB/CC2
- J2 pad B9A4: /VBUSB -> /ESP USB/VBUS
- J7 pad 1: PWR_RAW -> /5V_stable
- J8 pad 1: PWR_RAW -> /5V_stable
- P1 pad 2: Net-(Q6-D) -> Net-(Q10-S)
- Q3 pad 1: /USB_5V -> Net-(Q3-G)
- Q3 pad 2: Net-(Q3-S) -> GND
- Q3 pad 3: /VBATT -> /ESP USB/USB_SOURCE_EN
- Q6 pad 1: Net-(Q6-G) -> /USB_LC
- Q6 pad 2: GND -> /USB_HC
- Q6 pad 3: Net-(Q6-D) -> /VBATT
- R19 pad 1: /LEDSingleMid -> Net-(LED1---Pad3)
- R19 pad 2: Net-(D14-Pad2) -> GND
- R20 pad 1: Net-(LED1---Pad3) -> Net-(LED1---Pad1)
- R21 pad 1: Net-(LED1---Pad1) -> Net-(LED1---Pad2)
- R22 pad 1: Net-(LED1---Pad2) -> /LEDSingleMid
- R22 pad 2: GND -> Net-(D14-Pad2)
- R24 pad 1: GND -> /VBATT
- R24 pad 2: /USB_5V -> Net-(Q10-G)
- R41 pad 1: Net-(Q4-D) -> PWR_RAW
- R44 pad 1: /VBATT -> /BatteryVoltage
- R44 pad 2: Net-(Q4-G) -> GND
- R46 pad 1: /BatteryVoltage -> PWR_RAW
- R46 pad 2: GND -> Net-(U2-EN)
- R48 pad 1: Net-(Q6-G) -> /Power Input Managment/VIN
- R48 pad 2: /VBATT -> Net-(D9-C)
- R5 pad 1: Net-(J2-CC1) -> /ESP USB/VBUS
- R5 pad 2: GND -> Net-(U8-VBUS_DET)
- R54 pad 1: PWR_RAW -> +3.3V
- R54 pad 2: Net-(U2-EN) -> Net-(D1-Pad2)
- R6 pad 1: Net-(J2-CC2) -> /5V_stable
- R6 pad 2: GND -> /ESP USB/USB_ID
- U2 pad 1: Net-(U2-EN) -> GND
- U4 pad 4: /USB_5V -> /USB_LC
- U4 pad 8: /USB_5V -> /USB_LC
- U8 pad 1: PWR_RAW -> /ESP USB/CC1
- U8 pad 2: GND -> /ESP USB/CC2
- U8 pad 3: PWR_RAW -> GND
- U8 pad 5: +3.3V -> Net-(U8-VBUS_DET)
Routing:
- net PWR_RAW: track 358.9 -> 54.1 mm, vias 0 -> 2
- net /5V_stable: track 229.8 -> 467.5 mm
- net /USB_5V: track 172.4 -> 0.00 mm, vias 8 -> 0
- net /USB_HC: track 0.00 -> 113.7 mm
- net /USB_LC: track 0.00 -> 88.9 mm
- net GND: track 223.4 -> 151.3 mm
- net /VBUS: track 17.8 -> 88.9 mm, vias 2 -> 8
- net +3.3V: track 479.8 -> 526.1 mm, vias 9 -> 11
- net /Power Input Managment/VIN: track 0.00 -> 44.6 mm
- net /ESP USB/VBUS: track 0.00 -> 38.7 mm
- net /BatteryVoltage: track 87.4 -> 52.9 mm, vias 3 -> 1
- net Net-(Q11-S): track 0.00 -> 15.4 mm
- net /ESP USB/USB_SOURCE_EN: track 0.00 -> 15.2 mm
- net /Power Input Managment/OV1_EN_N: track 0.00 -> 13.8 mm
- net /GPIO41: track 209.5 -> 223.3 mm, vias 5 -> 4
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Other:
- outline, holes or cut-outs redrawn
- board text added: "Display (SPI2) Chip Select: 0 Data/Cmd: 45 Reset: 1 SPI_CLK: 46 SPI_MOSI: 3 SD Card (SPI3) Chip Select: 40 SPI_MOSI: 39 SPI_CLK: 38 SPI_MISO: 37 Minibadge A CLK: 13 IO2: 14 IO1: 15 (See I2C) Minibadge B CLK: 16 IO2: 17 IO1: 18 (See I2C)"
- board text added: "LED: 6 Addr LEDs: 7 Buzzer: 48 RGB LED Red: 2 Green: 4 Blue: 5 Buttons Left: 21 Right: 10 Down: 47 Up: 11 B: 33 A: 34 Joystick X axis: 8 Y axis: 9 Accelerometer Address: 0x1C Board Input Voltage VMain: 12"
- board text added: "USB-CDC-DRD"
- board text added: "USB_PWR_SRC"
- board text added: "VBAT 2.8-4.2V"
- board text added: "VERSION 4.1.0 JUL26"
- board text added: "VIN 2.8-16V"
- board text added: "VMain"
- board text removed: "AL"
- board text removed: "Bt_V"
- board text removed: "Display (SPI2) Chip Select: 0 Data/Command: 45 Reset: 1 SPI_CLK: 46 SPI_MOSI: 3 SD Card (SPI3) Chip Select: 40 SPI_MOSI: 39 SPI_CLK: 38 SPI_MISO: 37 Minibadge A CLK: 13 IO2: 14 IO1: 15 (See I2C) Minibadge B CLK: 16 IO2: 17 IO1: 18 (See I2C)"
- board text removed: "LED: 6 Addr LEDs: 7 Buzzer: 48 RGB LED Red: 2 Green: 4 Blue: 5 Buttons Left: 21 Right: 10 Down: 47 Up: 11 B: 33 A: 34 Joystick X axis: 8 Y axis: 9 Accelerometer Address: 0x1C Battery Voltage Bt_V: 12"
- board text removed: "USB-CDC"
- board text removed: "VERSION 4.0 FEB26"

Commit message: changed buzzer pot
Parts:
- removed R64: 330Ω, PCM_JLCPCB:R_0402
- removed RV1: 1000Ω, Potentiometer_THT:Potentiometer_Bourns_3296W_Vertical
- added R2: 3362P-1-501_C48997906, lcsc-lib:RES-ADJ-TH_3362P, F.Cu at (167.6, 80.8)
- added R60: 300Ω, PCM_JLCPCB:R_0402, F.Cu at (177.0, 74.1)
- moved Q5 8.10 mm to (163.7, 77.3), turned to 0 degrees
- moved R42 6.29 mm to (166.1, 77.7)
- moved BUZZER1 2.88 mm to (160.5, 82.8), turned to 90 degrees
Routing:
- net /BuzzerMid: track 77.7 -> 86.2 mm
- net Net-(BUZZER1-+): track 6.07 -> 11.8 mm
- net +3.3V: track 526.1 -> 523.5 mm
- net Net-(R2-Pad2): track 4.45 -> 2.27 mm
- net Net-(BUZZER1--): track 5.48 -> 3.57 mm
- net GND: vias 379 -> 386
