File: hardware v4.0/badge-esp32-s3/Charging.kicad_sch (KiCad schematic)
At the start: 29 parts, among them P1 PH-2A_C2319, P3 WJ124-3.81-2P, Q6 AO3424, Q8 HL2301A, Q9 AO3424, SW3 SK-22F18-G050, U4 TP4056, U5 TPS2121RUXR

Commit message: finished schematics and layout
Parts:
- removed C43: 470nF, PCM_JLCPCB:C_0402, symbol PCM_JLCPCB-Capacitors:0402,470nF
- removed D10, D15: BZX585-B10,115, lcsc-lib:SOD-523_L1.2-W0.8-LS1.6-RD, symbol lcsc-lib:BZX585-B10,115
- removed D11: B0520W, PCM_JLCPCB:D_SOD-123, symbol PCM_JLCPCB-Diodes:Schottky,B0520W
- removed Power1: SK-12F04-G050, lcsc-lib:SW-TH_G-SWITCH_SK-12F04-G050, symbol lcsc-lib:SK-12F04-G050
- removed Q6, Q9: AO3424, lcsc-lib:SC-59-3_L2.9-W1.6-P0.95-LS2.9-BR, symbol lcsc-lib:AO3424
- removed Q8: HL2301A, PCM_JLCPCB:Q_SOT-23, symbol PCM_JLCPCB-Transistors:PMOS,HL2301A
- removed R57: 220kΩ, PCM_JLCPCB:R_0402, symbol PCM_JLCPCB-Resistors:0402,220kΩ
- removed R58: 15kΩ, PCM_JLCPCB:R_0402, symbol PCM_JLCPCB-Resistors:0402,15kΩ
- removed R59, R60: 100Ω, PCM_JLCPCB:R_0402, symbol PCM_JLCPCB-Resistors:0402,100Ω
- removed R61: 75kΩ, PCM_JLCPCB:R_0402, symbol PCM_JLCPCB-Resistors:0402,75kΩ
- removed R63: 22kΩ, PCM_JLCPCB:R_0402, symbol PCM_JLCPCB-Resistors:0402,22kΩ
- removed SW3: SK-22F18-G050, lcsc-lib:SW-TH_SK-22F18-G050, symbol lcsc-lib:SK-22F18-G050
- added C41: 100nF, PCM_JLCPCB:C_0402, symbol PCM_JLCPCB-Capacitors:0402,100nF,(2)
- added D20, D21: BZT52-B5V1S, lcsc-lib:SOD-323_L1.8-W1.3-LS2.5-RD, symbol lcsc-lib:BZT52-B5V1S_R1_00001
- added D9: BZT52-B10S-PEC, lcsc-lib:SOD-323_L1.8-W1.3-LS2.5-RD-1, symbol lcsc-lib:BZT52-B10S-PEC
- added Q10, Q11: DMN3150L-7, lcsc-lib:SOT-23-3_L2.9-W1.6-P1.90-LS2.8-BR-CW, symbol lcsc-lib:DMN3150L-7
- added Q6: SI2301CDS-T1-GE3, lcsc-lib:SOT-23-3_L3.0-W1.7-P0.95-LS2.9-BR, symbol lcsc-lib:SI2301CDS-T1-GE3
- added R57: 68kΩ, PCM_JLCPCB:R_0402, symbol PCM_JLCPCB-Resistors:0402,68kΩ
- added R58: 47kΩ, PCM_JLCPCB:R_0402, symbol PCM_JLCPCB-Resistors:0402,47kΩ
- added R59: 1MΩ, PCM_JLCPCB:R_0402, symbol PCM_JLCPCB-Resistors:0402,1MΩ
- added R71: 470kΩ, PCM_JLCPCB:R_0402, symbol PCM_JLCPCB-Resistors:0402,470kΩ
- added SW10: SK22D02G5, lcsc-lib:SW-TH_SK22D02G5, symbol lcsc-lib:SK22D02G5
Connections:
- net PWR_2 is gone; now on net VIN: U5.2 (IN2)
- net USB_5V is gone; now on net USB_LC: C12.1, D12.2, U4.4 (VCC), U4.8 (CE)
- net GND: now also R56.2, C41.2, D20.2 (A), D21.2 (A), D9.2 (A), Q10.2 (D), Q11.2 (D), R58.2, SW10.3, SW10.4, SW10.7, SW10.8
- net VBATT: now also Q6.3 (D)
- net VIN: now also R59.1
- net at R48.2: now also D9.1 (C), Q11.1 (G)
- net at U5.5 (OV1): now also R62.1, D21.1 (K), R71.2; no longer R62.2
- net at P3.2: now also Q11.3 (S)
- net at U5.4 (OV2): now also D20.1 (K), R57.1, R59.2
- net at U5.11 (SS): now also C41.1
- net at R24.2: now also Q10.1 (G)
- net at P1.2: now also Q10.3 (S)
- net at U5.10 (ILM): now also R58.1
- net USB_LC: now reaches R56.1
- net USB_LC: now also Q6.1 (G)
- net PWR_1 renamed USB_HC
- net USB_HC: now also Q6.2 (S), R71.1; no longer R62.1
- new net OV1_EN_N: R62.2, SW10.2
- new net OV2_EN_N: R57.2, SW10.5
- no-connect marks 0 -> 2
Other:
- note added: "Current Limit: ~2.36A"
- note added: "Does not need gate protection diode as the voltage should not get that high on this source."
- note added: "Over Voltage: ~6V"
- note added: "Power EN"
- note added: "Power MUX"
- note added: "Universal External Voltage supply. Vin = 2.8V - 16V"
- note added: "lipo/lion charger and reverse polarity protection"
- note removed: "Current Limit: ~1.5A"
- note removed: "Over Voltage: ~5.8V"
- note removed: "Voltage ramp to 7.5ms @ 16V"
- moved on the sheet: C12, C13, C24, D12, P1, P3, R24, R25, R26, R48, R56, R62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

Commit message: changed PWR switch and current limit
Parts:
- removed R58: 47kΩ, PCM_JLCPCB:R_0402, symbol PCM_JLCPCB-Resistors:0402,47kΩ
- added R63: 39kΩ, PCM_JLCPCB:R_0402, symbol PCM_JLCPCB-Resistors:0402,39kΩ
- SW10: LCSC Part C22435631 -> C22435630
Connections:
- net GND: now also R63.2
- net at U5.10 (ILM): now also R63.1
Other:
- note added: "Current Limit: ~2.8A"
- note removed: "Current Limit: ~2.36A"
Changed lines of the file:
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@@
 		)
 	)
-	(text "Current Limit: ~2.36A"
+	(text "Current Limit: ~2.8A"
 		(exclude_from_sim no)
 		(at 247.65 129.794 0)
@@
 		(polyline
 			(pts
-				(xy 17.78 16.51) (xy 193.04 16.51) (xy 193.04 63.5) (xy 17.78 63.5)
+				(xy 17.78 69.85) (xy 127 69.85) (xy 127 120.65) (xy 17.78 120.65)
 			)
 			(stroke
@@
 		(polyline
 			(pts
-				(xy 17.78 69.85) (xy 127 69.85) (xy 127 120.65) (xy 17.78 120.65)
+				(xy 17.78 16.51) (xy 193.04 16.51) (xy 193.04 63.5) (xy 17.78 63.5)
 			)
 			(stroke
@@
 		(polyline
 			(pts
-				(xy 129.54 70.485) (xy 283.21 70.485) (xy 283.21 160.655) (xy 129.54 160.655)
+				(xy 17.78 127) (xy 127 127) (xy 127 185.42) (xy 17.78 185.42)
 			)
 			(stroke
@@
 		(polyline
 			(pts
-				(xy 17.78 127) (xy 127 127) (xy 127 185.42) (xy 17.78 185.42)
+				(xy 129.54 70.485) (xy 283.21 70.485) (xy 283.21 160.655) (xy 129.54 160.655)
 			)
 			(stroke
@@
 	)
 	(symbol
-		(lib_id "PCM_JLCPCB-Resistors:0402,47kΩ")
+		(lib_id "PCM_JLCPCB-Resistors:0402,39kΩ")
 		(at 246.38 134.62 0)
 		(unit 1)
@@
 		(dnp no)
 		(fields_autoplaced yes)
-		(property "Reference" "R58"
+		(property "Reference" "R63"
 			(at 248.92 134.6199 0)
 			(effects
@@
 			)
 		)
-		(property "Value" "47kΩ"
+		(property "Value" "39kΩ"
 			(at 246.38 134.62 90)
 			(do_not_autoplace yes)
@@
 			)
 		)
-		(property "Datasheet" "https://www.lcsc.com/datasheet/lcsc_datasheet_2206010100_UNI-ROYAL-Uniroyal-Elec-0402WGF4702TCE_C25792.pdf"
+		(property "Datasheet" "https://www.lcsc.com/datasheet/lcsc_datasheet_2206010100_UNI-ROYAL-Uniroyal-Elec-0402WGF3902TCE_C25783.pdf"
 			(at 246.38 134.62 0)
 			(effects
@@
 			)
 		)
-		(property "Description" "62.5mW Thick Film Resistors 50V ±100ppm/°C ±1% 47kΩ 0402 Chip Resistor - Surface Mount ROHS"
+		(property "Description" "62.5mW Thick Film Resistors 50V ±100ppm/°C ±1% 39kΩ 0402 Chip Resistor - Surface Mount ROHS"
 			(at 246.38 134.62 0)
 			(effects
@@
 			)
 		)
-		(property "LCSC" "C25792"
+		(property "LCSC" "C25783"
 			(at 246.38 134.62 0)
 			(effects
@@
 			)
 		)
-		(property "Stock" "1792808"
+		(property "Stock" "215714"
 			(at 246.38 134.62 0)
 			(effects
@@
 			)
 		)
-		(property "Class" "Basic Component"
+		(property "Class" "Preferred Component"
 			(at 246.38 134.62 0)
 			(effects
@@
 			)
 		)
-		(property "Part" "0402WGF4702TCE"
+		(property "Part" "0402WGF3902TCE"
 			(at 246.38 134.62 0)
 			(effects
@@
 			)
 		)
-		(property "Resistance" "47kΩ"
+		(property "Resistance" "39kΩ"
 			(at 246.38 134.62 0)
 			(effects
@@
 			(project ""
 				(path "/e2af9a6c-dbe9-4de2-9ba6-ea213a7300ec/9131a646-b9dc-4004-a7df-1b58b7ca0b9a"
-					(reference "R58")
+					(reference "R63")
 					(unit 1)
 				)
@@
 			)
 		)
-		(property "LCSC Part" "C22435631"
+		(property "LCSC Part" "C22435630"
 			(at 40.64 154.94 0)
 			(effects
