File: hardware v4.1.1/badge-esp32-s3/3-3V_delivery.kicad_sch (KiCad schematic)
At the start: 26 parts, among them U2 TPS630701RNMR, U9 AP63201WU-7

Commit message: fixed out of stock components
Parts:
- removed L3: XGL4020-152MEC, lcsc-lib:IND-SMD_L4.0-W4.0_XEL4020, symbol lcsc-lib:XGL4020-152MEC
- removed R64: 75kΩ, PCM_JLCPCB:R_0402, symbol PCM_JLCPCB-Resistors:0402,75kΩ
- added L4: FTC404020S1R5MGCA, lcsc-lib:IND-SMD_L4.1-W4.1_SPM40XX, symbol lcsc-lib:FTC404020S1R5MGCA
- added R64: 0Ω, PCM_JLCPCB:R_0402, symbol PCM_JLCPCB-Resistors:0402,0Ω
- C28, C29, C30, C31, C38, C40: Attrition Qty 8 -> (none); Capacitance 22uF -> (none); Category Capacitors,Multilayer Ceramic Capacitors MLCC - SMD/SMT -> (none); Class Basic Component -> (none); LCSC C45783 -> C296720; Manufacturer Samsung Electro-Mechanics -> (none); Minimum Qty 20 -> (none); Part CL21A226MAQNNNE -> (none); Price 0.027USD -> (none); Process SMT -> (none); Stock 6479946 -> (none); Temperature Coefficient X5R -> (none); Tolerance ±20% -> (none); Voltage Rated 25V -> (none)
- R19: now not fitted; now left out of the parts list
Connections:
- net VCC_3V3: now also R64.1
- net at R19.1, U9.1 (FB): now also R64.2
- net at U2.11 (L1): now also L4.1
- net at U2.9 (L2): now also L4.2

Commit message: changed 3.3V reg from adj to fixed
changed 3.3V reg from adj to fixed and reflexed that in the bom
Parts:
- U9: value AP63201WU-7 -> AP63203WU-7; LCSC Part C2071044 -> C780769; MPN AP63201WU-7 -> AP63203WU-7
Changed lines of the file:
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@@
 			)
 		)
-		(property "Value" "AP63201WU-7"
+		(property "Value" "AP63203WU-7"
 			(at 143.51 107.95 0)
 			(effects
@@
 			)
 		)
-		(property "MPN" "AP63201WU-7"
+		(property "MPN" "AP63203WU-7"
 			(at 143.51 133.35 0)
 			(effects
@@
 			)
 		)
-		(property "LCSC Part" "C2071044"
+		(property "LCSC Part" "C780769"
 			(at 143.51 135.89 0)
 			(effects
