File: hardware v4.1.1/badge-esp32-s3/usbc_esp_5v_v2_data.kicad_sch (KiCad schematic)
At the start: 23 parts, among them J2 Connector, USB-TYPE-C-16P, Q3 AP1606, U11 SY6288F1ABC, U12 SY6288F1ABC, U8 TUSB321AIRWBR

Commit message: fixed out of stock components
Parts:
- U11, U12: Alternate LCSC (none) -> C2687365; Notes (none) -> This alternate part is more complex and overkill for this s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
Changed lines of the file:
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@@
 		(polyline
 			(pts
-				(xy 17.78 19.05) (xy 172.72 19.05) (xy 172.72 68.58) (xy 17.78 68.58)
+				(xy 17.78 74.93) (xy 238.76 74.93) (xy 238.76 161.29) (xy 17.78 161.29)
 			)
 			(stroke
@@
 		(polyline
 			(pts
-				(xy 17.78 74.93) (xy 238.76 74.93) (xy 238.76 161.29) (xy 17.78 161.29)
+				(xy 17.78 19.05) (xy 172.72 19.05) (xy 172.72 68.58) (xy 17.78 68.58)
 			)
 			(stroke
@@
 			)
 		)
+		(property "Alternate LCSC" "C2687365"
+			(at 157.48 135.89 0)
+			(effects
+				(font
+					(size 1.27 1.27)
+				)
+				(hide yes)
+			)
+		)
+		(property "Notes" "This alternate part is more complex and overkill for this situation but will work as a drop in replacement. It also will see about a 4% higher current limit as it uses a different current limit equation."
+			(at 157.48 135.89 0)
+			(effects
+				(font
+					(size 1.27 1.27)
+				)
+				(hide yes)
+			)
+		)
 		(pin "4"
 		)
@@
 			(effects
 				(font
+					(size 1.27 1.27)
+				)
+				(hide yes)
+			)
+		)
+		(property "Alternate LCSC" "C2687365"
+			(at 157.48 85.09 0)
+			(effects
+				(font
+					(size 1.27 1.27)
+				)
+				(hide yes)
+			)
+		)
+		(property "Notes" "This alternate part is more complex and overkill for this situation but will work as a drop in replacement. It also will see about a 4% higher current limit as it uses a different current limit equation."
+			(at 157.48 85.09 0)
+			(effects
+				(font
